File: hardware/stm32/eeprom.sch (KiCad schematic (older format))
At the start: 1 part, among them U2 24LC512

Commit message: bluepill Schematics 0.99
Parts:
- added C2, C3: 100n, Capacitors_SMD:C_0805, symbol C_Small
- added J14: RTC, Pin_Headers:Pin_Header_Straight_1x06_Pitch2.54mm, symbol Conn_01x06
Connections:
- net +5V: now also C2.1, C3.1, J14.2 (Pin_2)
- net GND: now also C2.2, C3.2, J14.1 (Pin_1)
- net SCL: now also J14.4 (Pin_4)
- net SDA: now also J14.3 (Pin_3)
Changed lines of the file:
@@
 LIBS:power
 LIBS:device
+LIBS:switches
+LIBS:relays
+LIBS:motors
+LIBS:transistors
+LIBS:conn
 LIBS:linear
 LIBS:regul
+LIBS:74xx
+LIBS:cmos4000
 LIBS:adc-dac
 LIBS:memory
@@
 LIBS:atmel
 LIBS:contrib
+LIBS:valves
 LIBS:bluepill
 LIBS:Connector
@@
 	1    0    0    -1
 $EndComp
-Text HLabel 6600 3850 2    60   Output ~ 0
-SCL
-Text HLabel 6600 3750 2    60   BiDi ~ 0
-SDA
-Wire Wire Line
-	6200 3750 6600 3750
-Wire Wire Line
-	6200 3850 6600 3850
-$Comp
-L +5V #PWR01
+Text HLabel 7250 3850 2    60   Output ~ 0
+SCL
+Text HLabel 7250 3750 2    60   BiDi ~ 0
+SDA
+$Comp
+L +5V #PWR5
 U 1 1 5A5F3296
-P 5800 3300
-F 0 "#PWR01" H 5800 3150 50  0001 C CNN
-F 1 "+5V" H 5800 3440 50  0000 C CNN
-F 2 "" H 5800 3300 50  0001 C CNN
-F 3 "" H 5800 3300 50  0001 C CNN
-	1    5800 3300
-	1    0    0    -1
-$EndComp
-$Comp
-L GND #PWR02
+P 5800 3450
+F 0 "#PWR5" H 5800 3300 50  0001 C CNN
+F 1 "+5V" H 5800 3590 50  0000 C CNN
+F 2 "" H 5800 3450 50  0001 C CNN
+F 3 "" H 5800 3450 50  0001 C CNN
+	1    5800 3450
+	1    0    0    -1
+$EndComp
+$Comp
+L GND #PWR6
 U 1 1 5A5F32AC
 P 5800 4500
-F 0 "#PWR02" H 5800 4250 50  0001 C CNN
+F 0 "#PWR6" H 5800 4250 50  0001 C CNN
 F 1 "GND" H 5800 4350 50  0000 C CNN
 F 2 "" H 5800 4500 50  0001 C CNN
@@
 $EndComp
 Wire Wire Line
-	5800 3550 5800 3300
+	5800 3550 5800 3450
 Wire Wire Line
 	5800 4150 5800 4500
@@
 Wire Wire Line
 	6200 4250 6200 3950
+$Comp
+L Conn_01x06 J14
+U 1 1 5A604F2C
+P 6700 2950
+F 0 "J14" H 6700 3250 50  0000 C CNN
+F 1 "RTC" H 6700 2550 50  0000 C CNN
+F 2 "Pin_Headers:Pin_Header_Straight_1x06_Pitch2.54mm" H 6700 2950 50  0001 C CNN
+F 3 "" H 6700 2950 50  0001 C CNN
+	1    6700 2950
+	1    0    0    1
+$EndComp
+$Comp
+L GND #PWR8
+U 1 1 5A604F8F
+P 6450 3250
+F 0 "#PWR8" H 6450 3000 50  0001 C CNN
+F 1 "GND" H 6450 3100 50  0000 C CNN
+F 2 "" H 6450 3250 50  0001 C CNN
+F 3 "" H 6450 3250 50  0001 C CNN
+	1    6450 3250
+	1    0    0    -1
+$EndComp
+$Comp
+L C_Small C2
+U 1 1 5A604FD2
+P 5250 3000
+F 0 "C2" H 5260 3070 50  0000 L CNN
+F 1 "100n" H 5260 2920 50  0000 L CNN
+F 2 "Capacitors_SMD:C_0805" H 5250 3000 50  0001 C CNN
+F 3 "" H 5250 3000 50  0001 C CNN
+	1    5250 3000
+	1    0    0    -1
+$EndComp
+$Comp
+L +5V #PWR1
+U 1 1 5A605092
+P 5250 2800
+F 0 "#PWR1" H 5250 2650 50  0001 C CNN
+F 1 "+5V" H 5250 2940 50  0000 C CNN
+F 2 "" H 5250 2800 50  0001 C CNN
+F 3 "" H 5250 2800 50  0001 C CNN
+	1    5250 2800
+	1    0    0    -1
+$EndComp
+$Comp
+L GND #PWR2
+U 1 1 5A6050A6
+P 5250 3200
+F 0 "#PWR2" H 5250 2950 50  0001 C CNN
+F 1 "GND" H 5250 3050 50  0000 C CNN
+F 2 "" H 5250 3200 50  0001 C CNN
+F 3 "" H 5250 3200 50  0001 C CNN
+	1    5250 3200
+	1    0    0    -1
+$EndComp
+$Comp
+L +5V #PWR7
+U 1 1 5A6050C2
+P 6450 2550
+F 0 "#PWR7" H 6450 2400 50  0001 C CNN
+F 1 "+5V" H 6450 2690 50  0000 C CNN
+F 2 "" H 6450 2550 50  0001 C CNN
+F 3 "" H 6450 2550 50  0001 C CNN
+	1    6450 2550
+	1    0    0    -1
+$EndComp
+Wire Wire Line
+	6500 3150 6450 3150
+Wire Wire Line
+	6450 3150 6450 3250
+Wire Wire Line
+	6500 3050 6450 3050
+Wire Wire Line
+	6450 3050 6450 2550
+Wire Wire Line
+	5250 2800 5250 2900
+Wire Wire Line
+	5250 3100 5250 3200
+Wire Wire Line
+	6500 2950 6350 2950
+Wire Wire Line
+	6500 2850 6350 2850
+Wire Wire Line
+	6200 3750 6350 3750
+Wire Wire Line
+	6200 3850 6350 3850
+Wire Wire Line
+	7250 3750 7100 3750
+Wire Wire Line
+	7250 3850 7100 3850
+Text Label 7100 3750 2    60   ~ 0
+SDA
+Text Label 7100 3850 2    60   ~ 0
+SCL
+Text Label 6350 3750 0    60   ~ 0
+SDA
+Text Label 6350 3850 0    60   ~ 0
+SCL
+Text Label 6350 2950 2    60   ~ 0
+SDA
+Text Label 6350 2850 2    60   ~ 0
+SCL
+$Comp
+L C_Small C3
+U 1 1 5A605271
+P 5550 3000
+F 0 "C3" H 5560 3070 50  0000 L CNN
+F 1 "100n" H 5560 2920 50  0000 L CNN
+F 2 "Capacitors_SMD:C_0805" H 5550 3000 50  0001 C CNN
+F 3 "" H 5550 3000 50  0001 C CNN
+	1    5550 3000
+	1    0    0    -1
+$EndComp
+$Comp
+L +5V #PWR3
+U 1 1 5A605277
+P 5550 2800
+F 0 "#PWR3" H 5550 2650 50  0001 C CNN
+F 1 "+5V" H 5550 2940 50  0000 C CNN
+F 2 "" H 5550 2800 50  0001 C CNN
+F 3 "" H 5550 2800 50  0001 C CNN
+	1    5550 2800
+	1    0    0    -1
+$EndComp
+$Comp
+L GND #PWR4
+U 1 1 5A60527D
+P 5550 3200
+F 0 "#PWR4" H 5550 2950 50  0001 C CNN
+F 1 "GND" H 5550 3050 50  0000 C CNN
+F 2 "" H 5550 3200 50  0001 C CNN
+F 3 "" H 5550 3200 50  0001 C CNN
+	1    5550 3200
+	1    0    0    -1
+$EndComp
+Wire Wire Line
+	5550 2800 5550 2900
+Wire Wire Line
+	5550 3100 5550 3200
 $EndSCHEMATC

Commit message: bluepill: PCB 0.9
Parts:
- removed C2: 100n, Capacitors_SMD:C_0805, symbol C_Small
Changed lines of the file:
@@
 SDA
 $Comp
-L +5V #PWR01
+L +5V #PWR3
 U 1 1 5A5F3296
 P 5800 3450
-F 0 "#PWR01" H 5800 3300 50  0001 C CNN
+F 0 "#PWR3" H 5800 3300 50  0001 C CNN
 F 1 "+5V" H 5800 3590 50  0000 C CNN
 F 2 "" H 5800 3450 50  0001 C CNN
@@
 $EndComp
 $Comp
-L GND #PWR02
+L GND #PWR4
 U 1 1 5A5F32AC
 P 5800 4500
-F 0 "#PWR02" H 5800 4250 50  0001 C CNN
+F 0 "#PWR4" H 5800 4250 50  0001 C CNN
 F 1 "GND" H 5800 4350 50  0000 C CNN
 F 2 "" H 5800 4500 50  0001 C CNN
@@
 $EndComp
 $Comp
-L GND #PWR03
+L GND #PWR6
 U 1 1 5A604F8F
 P 6450 3250
-F 0 "#PWR03" H 6450 3000 50  0001 C CNN
+F 0 "#PWR6" H 6450 3000 50  0001 C CNN
 F 1 "GND" H 6450 3100 50  0000 C CNN
 F 2 "" H 6450 3250 50  0001 C CNN
@@
 $EndComp
 $Comp
-L C_Small C2
-U 1 1 5A604FD2
-P 5250 3000
-F 0 "C2" H 5260 3070 50  0000 L CNN
-F 1 "100n" H 5260 2920 50  0000 L CNN
-F 2 "Capacitors_SMD:C_0805" H 5250 3000 50  0001 C CNN
-F 3 "" H 5250 3000 50  0001 C CNN
-	1    5250 3000
-	1    0    0    -1
-$EndComp
-$Comp
-L +5V #PWR04
-U 1 1 5A605092
-P 5250 2800
-F 0 "#PWR04" H 5250 2650 50  0001 C CNN
-F 1 "+5V" H 5250 2940 50  0000 C CNN
-F 2 "" H 5250 2800 50  0001 C CNN
-F 3 "" H 5250 2800 50  0001 C CNN
-	1    5250 2800
-	1    0    0    -1
-$EndComp
-$Comp
-L GND #PWR05
-U 1 1 5A6050A6
-P 5250 3200
-F 0 "#PWR05" H 5250 2950 50  0001 C CNN
-F 1 "GND" H 5250 3050 50  0000 C CNN
-F 2 "" H 5250 3200 50  0001 C CNN
-F 3 "" H 5250 3200 50  0001 C CNN
-	1    5250 3200
-	1    0    0    -1
-$EndComp
-$Comp
-L +5V #PWR06
+L +5V #PWR5
 U 1 1 5A6050C2
 P 6450 2550
-F 0 "#PWR06" H 6450 2400 50  0001 C CNN
+F 0 "#PWR5" H 6450 2400 50  0001 C CNN
 F 1 "+5V" H 6450 2690 50  0000 C CNN
 F 2 "" H 6450 2550 50  0001 C CNN
@@
 Wire Wire Line
 	6450 3050 6450 2550
-Wire Wire Line
-	5250 2800 5250 2900
-Wire Wire Line
-	5250 3100 5250 3200
 Wire Wire Line
 	6500 2950 6350 2950
@@
 $EndComp
 $Comp
-L +5V #PWR07
+L +5V #PWR1
 U 1 1 5A605277
 P 5550 2800
-F 0 "#PWR07" H 5550 2650 50  0001 C CNN
+F 0 "#PWR1" H 5550 2650 50  0001 C CNN
 F 1 "+5V" H 5550 2940 50  0000 C CNN
 F 2 "" H 5550 2800 50  0001 C CNN
@@
 $EndComp
 $Comp
-L GND #PWR08
+L GND #PWR2
 U 1 1 5A60527D
 P 5550 3200
-F 0 "#PWR08" H 5550 2950 50  0001 C CNN
+F 0 "#PWR2" H 5550 2950 50  0001 C CNN
 F 1 "GND" H 5550 3050 50  0000 C CNN
 F 2 "" H 5550 3200 50  0001 C CNN
